Commit message: add base_footprint

File: src/auracle_description/urdf/robot_core.xacro (robot description, xacro)
@@ -33,4 +33,14 @@
         <color rgba="1 0 0 1"/>
     </material>
+    <!-- BASE FOOTPRINT: ground-projected frame, kept at true wheel-contact
+        height. This is the frame EKF/Nav2/SLAM should track — see ekf.yaml,
+        nav2_params.yaml, mapper_params_online_async.yaml. -->
+    <link name="base_footprint"/>
+    <joint name="base_footprint_joint" type="fixed">
+        <parent link="base_footprint"/>
+        <child link="base_link"/>
+        <!-- 0.0707 (wheel center drop from base_link) + 0.0239 (wheel_radius) -->
+        <origin xyz="0 0 0.0946" rpy="0 0 0"/>
+    </joint>
     <!-- BASE LINK -->
     <link name="base_link">
@@ -427,3 +437,25 @@
         <material>Gazebo/Blue</material>
     </gazebo>
+    <!-- Gazebo Sim/ODE does not support <mimic> constraints (see the
+        "Attempting to create a mimic constraint" warning at spawn time), so
+        left/right_wheel_one and left/right_wheel_three are un-driven, free
+        joints sitting in full-friction ground contact in sim. That's enough
+        drag from 4 wheels to stop 2 driven wheels from pivoting the chassis.
+        Cut their friction drastically so they can scrub/slide during turns. -->
+    <gazebo reference="left_wheel_one">
+        <mu1>0.01</mu1>
+        <mu2>0.01</mu2>
+    </gazebo>
+    <gazebo reference="left_wheel_three">
+        <mu1>0.01</mu1>
+        <mu2>0.01</mu2>
+    </gazebo>
+    <gazebo reference="right_wheel_one">
+        <mu1>0.01</mu1>
+        <mu2>0.01</mu2>
+    </gazebo>
+    <gazebo reference="right_wheel_three">
+        <mu1>0.01</mu1>
+        <mu2>0.01</mu2>
+    </gazebo>
 </robot>

Commit message: fix turning on gazebo

File: src/auracle_description/urdf/robot_core.xacro (robot description, xacro)
@@ -11,5 +11,4 @@
     <xacro:property name="tilted_link" value="0.1"/>
     <xacro:property name="rocker_mass" value="0.5"/>
-    <!-- Measured from emmanuel-assembly.stp tire rolling-surface cylinder (was 0.033) -->
     <xacro:property name="wheel_radius" value="0.0239"/>
     <xacro:property name="wheel_thickness" value="0.026"/>
@@ -33,12 +32,9 @@
         <color rgba="1 0 0 1"/>
     </material>
-    <!-- BASE FOOTPRINT: ground-projected frame, kept at true wheel-contact
-        height. This is the frame EKF/Nav2/SLAM should track — see ekf.yaml,
-        nav2_params.yaml, mapper_params_online_async.yaml. -->
+    <!-- BASE FOOTPRINT: ground-projected frame -->
     <link name="base_footprint"/>
     <joint name="base_footprint_joint" type="fixed">
         <parent link="base_footprint"/>
         <child link="base_link"/>
-        <!-- 0.0707 (wheel center drop from base_link) + 0.0239 (wheel_radius) -->
         <origin xyz="0 0 0.0946" rpy="0 0 0"/>
     </joint>
@@ -73,5 +69,5 @@
         <material>Gazebo/Orange</material>
     </gazebo>
- <!-- LEFT WHEEL ROCKER LINK -->
+    <!-- LEFT WHEEL ROCKER LINK -->
     <joint name="left_wheel_rocker_joint" type="fixed">
         <parent link="base_link"/>
@@ -145,9 +141,5 @@
         </xacro:inertial_box>
     </link>
-    <!-- LEFT WHEEL 1 -->
-    <!-- Not wired to ros2_control (only left_wheel_two_joint has a hardware
-         interface/encoder) - mimics left_wheel_two_joint so joint_state_publisher
-         (with use_mimic_tags) can still compute a valid rotation/TF for it instead
-         of it sitting frozen with no transform at all. -->
+    <!-- LEFT WHEEL 1 (Unactuated Front) -->
     <joint name="left_wheel_one_joint" type="continuous">
         <parent link="tilted_two_link"/>
@@ -176,5 +168,5 @@
         <material>Gazebo/Blue</material>
     </gazebo>
-    <!-- TILTED LINK6 -->
+    <!-- TILTED LINK3 -->
     <joint name="tilted_three_joint" type="fixed">
         <parent link="left_rocker"/>
@@ -200,7 +192,5 @@
         </xacro:inertial_box>
     </link>
-    <!-- LEFT WHEEL 3 -->
-    <!-- Not wired to ros2_control - mimics left_wheel_two_joint, same reasoning
-         as left_wheel_one_joint above. -->
+    <!-- LEFT WHEEL 3 (Unactuated Rear) -->
     <joint name="left_wheel_three_joint" type="continuous">
         <parent link="tilted_three_link"/>
@@ -229,5 +219,5 @@
         <material>Gazebo/Blue</material>
     </gazebo>
-     <!-- LEFT WHEEL 2 -->
+    <!-- LEFT WHEEL 2 (Driven Middle - Notice the collision radius bump) -->
     <joint name="left_wheel_two_joint" type="continuous">
         <parent link="tilted_link"/>
@@ -245,5 +235,5 @@
         <collision>
             <geometry>
-                <sphere radius="${wheel_radius}"/>
+                <sphere radius="${wheel_radius + 0.002}"/>
             </geometry>
         </collision>
@@ -279,5 +269,5 @@
         </xacro:inertial_box>
     </link>
-    <!-- TILTED LINK 1-->
+    <!-- TILTED LINK 1 -->
     <joint name="tilted_joint_two" type="fixed">
         <parent link="right_rocker"/>
@@ -327,9 +317,5 @@
         </xacro:inertial_box>
     </link>
-    <!-- RIGHT WHEEL 1 -->
-    <!-- Not wired to ros2_control (only right_wheel_two_joint has a hardware
-         interface/encoder) - mimics right_wheel_two_joint so joint_state_publisher
-         (with use_mimic_tags) can still compute a valid rotation/TF for it instead
-         of it sitting frozen with no transform at all. -->
+    <!-- RIGHT WHEEL 1 (Unactuated Front) -->
     <joint name="right_wheel_one_joint" type="continuous">
         <parent link="tilted_two_link_two"/>
@@ -359,5 +345,5 @@
     </gazebo>
     <!-- TILTED LINK3 -->
-     <joint name="tilted_two_joint_three" type="fixed">
+    <joint name="tilted_two_joint_three" type="fixed">
         <parent link="right_rocker"/>
         <child link="tilted_two_link_three"/>
@@ -382,7 +368,5 @@
         </xacro:inertial_box>
     </link>
-    <!-- RIGHT WHEEL 3 -->
-    <!-- Not wired to ros2_control - mimics right_wheel_two_joint, same reasoning
-         as right_wheel_one_joint above. -->
+    <!-- RIGHT WHEEL 3 (Unactuated Rear) -->
     <joint name="right_wheel_three_joint" type="continuous">
         <parent link="tilted_two_link_three"/>
@@ -411,5 +395,5 @@
         <material>Gazebo/Blue</material>
     </gazebo>
-     <!-- RIGHT WHEEL 2 -->
+    <!-- RIGHT WHEEL 2 (Driven Middle - Notice the collision radius bump) -->
     <joint name="right_wheel_two_joint" type="continuous">
         <parent link="tilted_link_two"/>
@@ -427,5 +411,5 @@
         <collision>
             <geometry>
-                <sphere radius="${wheel_radius}"/>
+                <sphere radius="${wheel_radius + 0.002}"/>
             </geometry>
         </collision>
@@ -437,10 +421,5 @@
         <material>Gazebo/Blue</material>
     </gazebo>
-    <!-- Gazebo Sim/ODE does not support <mimic> constraints (see the
-        "Attempting to create a mimic constraint" warning at spawn time), so
-        left/right_wheel_one and left/right_wheel_three are un-driven, free
-        joints sitting in full-friction ground contact in sim. That's enough
-        drag from 4 wheels to stop 2 driven wheels from pivoting the chassis.
-        Cut their friction drastically so they can scrub/slide during turns. -->
+    <!-- Gazebo Friction Overrides for the 4 outer unactuated wheels -->
     <gazebo reference="left_wheel_one">
         <mu1>0.01</mu1>

Commit message: update nav2 to use updated params

File: src/auracle_description/urdf/robot_core.xacro (robot description, xacro)
@@ -14,10 +14,9 @@
     <xacro:property name="wheel_thickness" value="0.026"/>
     <xacro:property name="wheel_mass" value="0.05"/>
-    <xacro:property name="wheel_offset_x" value="0.226"/>
-    <xacro:property name="wheel_offset_y" value="0.1485"/>
-    <xacro:property name="wheel_offset_z" value="0.01"/>
-    <material name="white">
-        <color rgba="1 1 1 1" />
+    <xacro:property name="camera_size" value="0.02"/>
+    <material name="red">
+        <color rgba="1 0 0 1"/>
     </material>
+    <joint name="camera_joint" type="fixed">
     <material name="orange">
         <color rgba="1 0.3 0.1 1"/>
@@ -29,7 +28,4 @@
         <color rgba="0 0 0 1"/>
     </material>
-    <material name="red">
-        <color rgba="1 0 0 1"/>
-    </material>
     <!-- BASE FOOTPRINT: ground-projected frame -->
     <link name="base_footprint"/>
@@ -141,5 +137,5 @@
         </xacro:inertial_box>
     </link>
-    <!-- LEFT WHEEL 1 (Unactuated Front) -->
+    <!-- LEFT WHEEL 1 (Unactuated Front - Mimic removed for Gazebo stability) -->
     <joint name="left_wheel_one_joint" type="continuous">
         <parent link="tilted_two_link"/>
@@ -147,5 +143,4 @@
         <origin xyz="0 0 ${-tilted_link}" rpy="0 ${pi/2} 0" />
         <axis xyz="0 0 1"/>
-        <mimic joint="left_wheel_two_joint" multiplier="1.0" offset="0.0"/>
     </joint>
     <link name="left_wheel_one">
@@ -192,5 +187,5 @@
         </xacro:inertial_box>
     </link>
-    <!-- LEFT WHEEL 3 (Unactuated Rear) -->
+    <!-- LEFT WHEEL 3 (Unactuated Rear - Mimic removed for Gazebo stability) -->
     <joint name="left_wheel_three_joint" type="continuous">
         <parent link="tilted_three_link"/>
@@ -198,5 +193,4 @@
         <origin xyz="0 0 ${-tilted_link}" rpy="0 ${pi/2} 0" />
         <axis xyz="0 0 1"/>
-        <mimic joint="left_wheel_two_joint" multiplier="1.0" offset="0.0"/>
     </joint>
     <link name="left_wheel_three">
@@ -219,5 +213,5 @@
         <material>Gazebo/Blue</material>
     </gazebo>
-    <!-- LEFT WHEEL 2 (Driven Middle - Notice the collision radius bump) -->
+    <!-- LEFT WHEEL 2 (Driven Middle) -->
     <joint name="left_wheel_two_joint" type="continuous">
         <parent link="tilted_link"/>
@@ -235,5 +229,5 @@
         <collision>
             <geometry>
-                <sphere radius="${wheel_radius + 0.002}"/>
+                <sphere radius="${wheel_radius}"/>
             </geometry>
         </collision>
@@ -317,5 +311,5 @@
         </xacro:inertial_box>
     </link>
-    <!-- RIGHT WHEEL 1 (Unactuated Front) -->
+    <!-- RIGHT WHEEL 1 (Unactuated Front - Mimic removed) -->
     <joint name="right_wheel_one_joint" type="continuous">
         <parent link="tilted_two_link_two"/>
@@ -323,5 +317,4 @@
         <origin xyz="0 0 ${-tilted_link}" rpy="0 ${pi/2} 0" />
         <axis xyz="0 0 1"/>
-        <mimic joint="right_wheel_two_joint" multiplier="1.0" offset="0.0"/>
     </joint>
     <link name="right_wheel_one">
@@ -368,5 +361,5 @@
         </xacro:inertial_box>
     </link>
-    <!-- RIGHT WHEEL 3 (Unactuated Rear) -->
+    <!-- RIGHT WHEEL 3 (Unactuated Rear - Mimic removed) -->
     <joint name="right_wheel_three_joint" type="continuous">
         <parent link="tilted_two_link_three"/>
@@ -374,5 +367,4 @@
         <origin xyz="0 0 ${-tilted_link}" rpy="0 ${pi/2} 0" />
         <axis xyz="0 0 1"/>
-        <mimic joint="right_wheel_two_joint" multiplier="1.0" offset="0.0"/>
     </joint>
     <link name="right_wheel_three">
@@ -395,5 +387,5 @@
         <material>Gazebo/Blue</material>
     </gazebo>
-    <!-- RIGHT WHEEL 2 (Driven Middle - Notice the collision radius bump) -->
+    <!-- RIGHT WHEEL 2 (Driven Middle) -->
     <joint name="right_wheel_two_joint" type="continuous">
         <parent link="tilted_link_two"/>
@@ -411,5 +403,5 @@
         <collision>
             <geometry>
-                <sphere radius="${wheel_radius + 0.002}"/>
+                <sphere radius="${wheel_radius}"/>
             </geometry>
         </collision>
@@ -421,5 +413,5 @@
         <material>Gazebo/Blue</material>
     </gazebo>
-    <!-- Gazebo Friction Overrides for the 4 outer unactuated wheels -->
+    <!-- Gazebo Friction Overrides: Allows the 4 outer wheels to scrub/slide laterally -->
     <gazebo reference="left_wheel_one">
         <mu1>0.01</mu1>

Commit message: change rocker joints to revolute

File: src/auracle_description/urdf/robot_core.xacro (robot description, xacro)
@@ -57,8 +57,21 @@
         <material>Gazebo/Orange</material>
     </gazebo>
-    <joint name="left_wheel_rocker_joint" type="fixed">
+    <!-- Rocker-to-chassis pivot. This has to be a real joint, not fixed:
+         it's the main degree of freedom that lets the whole rocker arm
+         (and everything hanging off it) rock forward/back as the wheels
+         cross terrain, instead of forcing the chassis to satisfy an
+         over-constrained rigid geometry. Passive (no actuator, not in
+         ros2_control) - it's driven purely by ground contact forces, with
+         damping/friction added just for numerical settling. Axis "1 0 0"
+         here is expressed in this joint's own (already rotated by the
+         rpy below) frame, and corresponds to the robot's lateral/pitch
+         axis - the correct axis for a suspension arm to rock about. -->
+    <joint name="left_wheel_rocker_joint" type="revolute">
         <parent link="base_link"/>
         <child link="left_rocker"/>
         <origin xyz="${chassis_length/2} ${chassis_width/2+rocker_width/2} 0" rpy="0 0 ${pi/2}" />
+        <axis xyz="1 0 0"/>
+        <limit lower="-0.6" upper="0.6" effort="50" velocity="5"/>
+        <dynamics damping="2.0" friction="0.1"/>
     </joint>
     <link name="left_rocker">
@@ -103,8 +116,27 @@
         </xacro:inertial_box>
     </link>
+    <!-- Bogie pivot: on a real rocker-bogie, the two rear wheels per side
+         don't bolt straight onto the rocker - they hang off a small bogie
+         arm that itself pivots on the rocker, so those two wheels
+         equalize load on their own instead of forcing the rocker (and the
+         chassis above it) to twist to reach them both. Passive, same
+         reasoning as the rocker-to-chassis joint above. -->
+    <joint name="left_bogie_joint" type="revolute">
+        <parent link="left_rocker"/>
+        <child link="left_bogie"/>
+        <origin xyz="0 ${-rocker_length/2} 0" rpy="0 0 0" />
+        <axis xyz="1 0 0"/>
+        <limit lower="-0.4" upper="0.4" effort="50" velocity="5"/>
+        <dynamics damping="1.0" friction="0.1"/>
+    </joint>
+    <link name="left_bogie">
+        <xacro:inertial_box mass="0.05" x="0.02" y="0.02" z="0.02">
+            <origin xyz="0 0 0" rpy="0 0 0"/>
+        </xacro:inertial_box>
+    </link>
     <joint name="tilted_two_joint" type="fixed">
-        <parent link="left_rocker"/>
+        <parent link="left_bogie"/>
         <child link="tilted_two_link"/>
-        <origin xyz="0 ${-rocker_length/2} 0" rpy="${-pi/4} 0 0" />
+        <origin xyz="0 0 0" rpy="${-pi/4} 0 0" />
     </joint>
     <link name="tilted_two_link">
@@ -152,7 +184,7 @@
     </gazebo>
     <joint name="tilted_three_joint" type="fixed">
-        <parent link="left_rocker"/>
+        <parent link="left_bogie"/>
         <child link="tilted_three_link"/>
-        <origin xyz="0 ${-rocker_length/2} 0" rpy="${pi/4} 0 0" />
+        <origin xyz="0 0 0" rpy="${pi/4} 0 0" />
     </joint>
     <link name="tilted_three_link">
@@ -224,8 +256,11 @@
         <material>Gazebo/Blue</material>
     </gazebo>
-    <joint name="right_wheel_rocker_joint" type="fixed">
+    <joint name="right_wheel_rocker_joint" type="revolute">
         <parent link="base_link"/>
         <child link="right_rocker"/>
         <origin xyz="${chassis_length/2} ${-chassis_width/2-rocker_width/2} 0" rpy="0 0 ${pi/2}" />
+        <axis xyz="1 0 0"/>
+        <limit lower="-0.6" upper="0.6" effort="50" velocity="5"/>
+        <dynamics damping="2.0" friction="0.1"/>
     </joint>
     <link name="right_rocker">
@@ -270,8 +305,21 @@
         </xacro:inertial_box>
     </link>
+    <joint name="right_bogie_joint" type="revolute">
+        <parent link="right_rocker"/>
+        <child link="right_bogie"/>
+        <origin xyz="0 ${-rocker_length/2} 0" rpy="0 0 0" />
+        <axis xyz="1 0 0"/>
+        <limit lower="-0.4" upper="0.4" effort="50" velocity="5"/>
+        <dynamics damping="1.0" friction="0.1"/>
+    </joint>
+    <link name="right_bogie">
+        <xacro:inertial_box mass="0.05" x="0.02" y="0.02" z="0.02">
+            <origin xyz="0 0 0" rpy="0 0 0"/>
+        </xacro:inertial_box>
+    </link>
     <joint name="tilted_two_joint_two" type="fixed">
-        <parent link="right_rocker"/>
+        <parent link="right_bogie"/>
         <child link="tilted_two_link_two"/>
-        <origin xyz="0 ${-rocker_length/2} 0" rpy="${-pi/4} 0 0" />
+        <origin xyz="0 0 0" rpy="${-pi/4} 0 0" />
     </joint>
     <link name="tilted_two_link_two">
@@ -319,7 +367,7 @@
     </gazebo>
     <joint name="tilted_two_joint_three" type="fixed">
-        <parent link="right_rocker"/>
+        <parent link="right_bogie"/>
         <child link="tilted_two_link_three"/>
-        <origin xyz="0 ${-rocker_length/2} 0" rpy="${pi/4} 0 0" />
+        <origin xyz="0 0 0" rpy="${pi/4} 0 0" />
     </joint>
     <link name="tilted_two_link_three">

Commit message: update robot_core

File: src/auracle_description/urdf/robot_core.xacro (robot description, xacro)
@@ -106,12 +106,17 @@
             <material name="black"/>
         </visual>
-        <collision>
-            <origin xyz="${rocker_length/2} 0 ${rocker_height/2}"/>
-            <geometry>
-                <box size="${rocker_length} ${rocker_width} ${rocker_height}"/>
-            </geometry>
-        </collision>
-        <xacro:inertial_box mass="${rocker_mass}" x="${rocker_length}" y="${rocker_width}" z="${rocker_height}">
-            <origin xyz="${rocker_length/2} 0 ${rocker_height/2}" rpy="0 0 0"/>
+        <!-- Was a copy-paste of left_rocker's full 0.13x0.02x0.2 collision
+             box, sitting at an offset that doesn't match this link's own
+             (much smaller, 0.1x0.02x0.025) visual at all - a phantom
+             collision volume trailing off of this strut. Now matches the
+             visual exactly. -->
+        <collision>
+            <origin xyz="0 0 -${tilted_link/2}" rpy="0 ${pi/2} 0"/>
+            <geometry>
+                <box size="${tilted_link} ${rocker_width} 0.025"/>
+            </geometry>
+        </collision>
+        <xacro:inertial_box mass="${rocker_mass}" x="${tilted_link}" y="${rocker_width}" z="0.025">
+            <origin xyz="0 0 -${tilted_link/2}" rpy="0 ${pi/2} 0"/>
         </xacro:inertial_box>
     </link>
@@ -149,11 +154,11 @@
         </visual>
         <collision>
-            <origin xyz="${rocker_length/2} 0 ${rocker_height/2}"/>
-            <geometry>
-                <box size="${rocker_length} ${rocker_width} ${rocker_height}"/>
-            </geometry>
-        </collision>
-        <xacro:inertial_box mass="${rocker_mass}" x="${rocker_length}" y="${rocker_width}" z="${rocker_height}">
-            <origin xyz="${rocker_length/2} 0 ${rocker_height/2}" rpy="0 0 0"/>
+            <origin xyz="0 0 -${tilted_link/2}" rpy="0 ${pi/2} 0"/>
+            <geometry>
+                <box size="${tilted_link} ${rocker_width} 0.025"/>
+            </geometry>
+        </collision>
+        <xacro:inertial_box mass="${rocker_mass}" x="${tilted_link}" y="${rocker_width}" z="0.025">
+            <origin xyz="0 0 -${tilted_link/2}" rpy="0 ${pi/2} 0"/>
         </xacro:inertial_box>
     </link>
@@ -197,11 +202,11 @@
         </visual>
         <collision>
-            <origin xyz="${rocker_length/2} 0 ${rocker_height/2}"/>
-            <geometry>
-                <box size="${rocker_length} ${rocker_width} ${rocker_height}"/>
-            </geometry>
-        </collision>
-        <xacro:inertial_box mass="${rocker_mass}" x="${rocker_length}" y="${rocker_width}" z="${rocker_height}">
-            <origin xyz="${rocker_length/2} 0 ${rocker_height/2}" rpy="0 0 0"/>
+            <origin xyz="0 0 -${tilted_link/2}" rpy="0 ${pi/2} 0"/>
+            <geometry>
+                <box size="${tilted_link} ${rocker_width} 0.025"/>
+            </geometry>
+        </collision>
+        <xacro:inertial_box mass="${rocker_mass}" x="${tilted_link}" y="${rocker_width}" z="0.025">
+            <origin xyz="0 0 -${tilted_link/2}" rpy="0 ${pi/2} 0"/>
         </xacro:inertial_box>
     </link>
@@ -296,11 +301,11 @@
         </visual>
         <collision>
-            <origin xyz="${rocker_length/2} 0 ${rocker_height/2}"/>
-            <geometry>
-                <box size="${rocker_length} ${rocker_width} ${rocker_height}"/>
-            </geometry>
-        </collision>
-        <xacro:inertial_box mass="${rocker_mass}" x="${rocker_length}" y="${rocker_width}" z="${rocker_height}">
-            <origin xyz="${rocker_length/2} 0 ${rocker_height/2}" rpy="0 0 0"/>
+            <origin xyz="0 0 -${tilted_link/2}" rpy="0 ${pi/2} 0"/>
+            <geometry>
+                <box size="${tilted_link} ${rocker_width} 0.025"/>
+            </geometry>
+        </collision>
+        <xacro:inertial_box mass="${rocker_mass}" x="${tilted_link}" y="${rocker_width}" z="0.025">
+            <origin xyz="0 0 -${tilted_link/2}" rpy="0 ${pi/2} 0"/>
         </xacro:inertial_box>
     </link>
@@ -332,11 +337,11 @@
         </visual>
         <collision>
-            <origin xyz="${rocker_length/2} 0 ${rocker_height/2}"/>
-            <geometry>
-                <box size="${rocker_length} ${rocker_width} ${rocker_height}"/>
-            </geometry>
-        </collision>
-        <xacro:inertial_box mass="${rocker_mass}" x="${rocker_length}" y="${rocker_width}" z="${rocker_height}">
-            <origin xyz="${rocker_length/2} 0 ${rocker_height/2}" rpy="0 0 0"/>
+            <origin xyz="0 0 -${tilted_link/2}" rpy="0 ${pi/2} 0"/>
+            <geometry>
+                <box size="${tilted_link} ${rocker_width} 0.025"/>
+            </geometry>
+        </collision>
+        <xacro:inertial_box mass="${rocker_mass}" x="${tilted_link}" y="${rocker_width}" z="0.025">
+            <origin xyz="0 0 -${tilted_link/2}" rpy="0 ${pi/2} 0"/>
         </xacro:inertial_box>
     </link>
@@ -380,11 +385,11 @@
         </visual>
         <collision>
-            <origin xyz="${rocker_length/2} 0 ${rocker_height/2}"/>
-            <geometry>
-                <box size="${rocker_length} ${rocker_width} ${rocker_height}"/>
-            </geometry>
-        </collision>
-        <xacro:inertial_box mass="${rocker_mass}" x="${rocker_length}" y="${rocker_width}" z="${rocker_height}">
-            <origin xyz="${rocker_length/2} 0 ${rocker_height/2}" rpy="0 0 0"/>
+            <origin xyz="0 0 -${tilted_link/2}" rpy="0 ${pi/2} 0"/>
+            <geometry>
+                <box size="${tilted_link} ${rocker_width} 0.025"/>
+            </geometry>
+        </collision>
+        <xacro:inertial_box mass="${rocker_mass}" x="${tilted_link}" y="${rocker_width}" z="0.025">
+            <origin xyz="0 0 -${tilted_link/2}" rpy="0 ${pi/2} 0"/>
         </xacro:inertial_box>
     </link>
