Commit message: improve turning in gazebo

File: src/auracle_description/urdf/camera.xacro (robot description, xacro)
@@ -2,4 +2,7 @@
 <robot xmlns:xacro="http://www.ros.org/wiki/xacro" >
     <xacro:property name="camera_size" value="0.02"/>
+    <material name="red">
+        <color rgba="1 0 0 1"/>
+    </material>
     <joint name="camera_joint" type="fixed">
         <parent link="chassis"/>

File: src/auracle_description/urdf/robot_core.xacro (robot description, xacro)
@@ -14,9 +14,4 @@
     <xacro:property name="wheel_thickness" value="0.026"/>
     <xacro:property name="wheel_mass" value="0.05"/>
-    <xacro:property name="camera_size" value="0.02"/>
-    <material name="red">
-        <color rgba="1 0 0 1"/>
-    </material>
-    <joint name="camera_joint" type="fixed">
     <material name="orange">
         <color rgba="1 0.3 0.1 1"/>
@@ -28,5 +23,4 @@
         <color rgba="0 0 0 1"/>
     </material>
-    <!-- BASE FOOTPRINT: ground-projected frame -->
     <link name="base_footprint"/>
     <joint name="base_footprint_joint" type="fixed">
@@ -35,8 +29,6 @@
         <origin xyz="0 0 0.0946" rpy="0 0 0"/>
     </joint>
-    <!-- BASE LINK -->
     <link name="base_link">
     </link>
-    <!-- CHASSIS LINK -->
     <joint name="chassis_joint" type="fixed">
         <parent link="base_link"/>
@@ -65,5 +57,4 @@
         <material>Gazebo/Orange</material>
     </gazebo>
-    <!-- LEFT WHEEL ROCKER LINK -->
     <joint name="left_wheel_rocker_joint" type="fixed">
         <parent link="base_link"/>
@@ -89,5 +80,4 @@
         </xacro:inertial_box>
     </link>
-    <!-- TILTED LINK -->
     <joint name="tilted_joint" type="fixed">
         <parent link="left_rocker"/>
@@ -113,5 +103,4 @@
         </xacro:inertial_box>
     </link>
-    <!-- TILTED LINK2 -->
     <joint name="tilted_two_joint" type="fixed">
         <parent link="left_rocker"/>
@@ -137,9 +126,8 @@
         </xacro:inertial_box>
     </link>
-    <!-- LEFT WHEEL 1 (Unactuated Front - Mimic removed for Gazebo stability) -->
     <joint name="left_wheel_one_joint" type="continuous">
         <parent link="tilted_two_link"/>
         <child link="left_wheel_one"/>
-        <origin xyz="0 0 ${-tilted_link}" rpy="0 ${pi/2} 0" />
+        <origin xyz="0 0 ${-tilted_link + 0.002}" rpy="0 ${pi/2} 0" />
         <axis xyz="0 0 1"/>
     </joint>
@@ -163,5 +151,4 @@
         <material>Gazebo/Blue</material>
     </gazebo>
-    <!-- TILTED LINK3 -->
     <joint name="tilted_three_joint" type="fixed">
         <parent link="left_rocker"/>
@@ -187,9 +174,8 @@
         </xacro:inertial_box>
     </link>
-    <!-- LEFT WHEEL 3 (Unactuated Rear - Mimic removed for Gazebo stability) -->
     <joint name="left_wheel_three_joint" type="continuous">
         <parent link="tilted_three_link"/>
         <child link="left_wheel_three"/>
-        <origin xyz="0 0 ${-tilted_link}" rpy="0 ${pi/2} 0" />
+        <origin xyz="0 0 ${-tilted_link + 0.002}" rpy="0 ${pi/2} 0" />
         <axis xyz="0 0 1"/>
     </joint>
@@ -213,5 +199,4 @@
         <material>Gazebo/Blue</material>
     </gazebo>
-    <!-- LEFT WHEEL 2 (Driven Middle) -->
     <joint name="left_wheel_two_joint" type="continuous">
         <parent link="tilted_link"/>
@@ -239,5 +224,4 @@
         <material>Gazebo/Blue</material>
     </gazebo>
-    <!-- RIGHT WHEEL ROCKER LINK -->
     <joint name="right_wheel_rocker_joint" type="fixed">
         <parent link="base_link"/>
@@ -263,5 +247,4 @@
         </xacro:inertial_box>
     </link>
-    <!-- TILTED LINK 1 -->
     <joint name="tilted_joint_two" type="fixed">
         <parent link="right_rocker"/>
@@ -287,5 +270,4 @@
         </xacro:inertial_box>
     </link>
-    <!-- TILTED LINK2 -->
     <joint name="tilted_two_joint_two" type="fixed">
         <parent link="right_rocker"/>
@@ -311,9 +293,8 @@
         </xacro:inertial_box>
     </link>
-    <!-- RIGHT WHEEL 1 (Unactuated Front - Mimic removed) -->
     <joint name="right_wheel_one_joint" type="continuous">
         <parent link="tilted_two_link_two"/>
         <child link="right_wheel_one"/>
-        <origin xyz="0 0 ${-tilted_link}" rpy="0 ${pi/2} 0" />
+        <origin xyz="0 0 ${-tilted_link + 0.002}" rpy="0 ${pi/2} 0" />
         <axis xyz="0 0 1"/>
     </joint>
@@ -337,5 +318,4 @@
         <material>Gazebo/Blue</material>
     </gazebo>
-    <!-- TILTED LINK3 -->
     <joint name="tilted_two_joint_three" type="fixed">
         <parent link="right_rocker"/>
@@ -361,9 +341,8 @@
         </xacro:inertial_box>
     </link>
-    <!-- RIGHT WHEEL 3 (Unactuated Rear - Mimic removed) -->
     <joint name="right_wheel_three_joint" type="continuous">
         <parent link="tilted_two_link_three"/>
         <child link="right_wheel_three"/>
-        <origin xyz="0 0 ${-tilted_link}" rpy="0 ${pi/2} 0" />
+        <origin xyz="0 0 ${-tilted_link + 0.002}" rpy="0 ${pi/2} 0" />
         <axis xyz="0 0 1"/>
     </joint>
@@ -387,5 +366,4 @@
         <material>Gazebo/Blue</material>
     </gazebo>
-    <!-- RIGHT WHEEL 2 (Driven Middle) -->
     <joint name="right_wheel_two_joint" type="continuous">
         <parent link="tilted_link_two"/>
@@ -413,5 +391,4 @@
         <material>Gazebo/Blue</material>
     </gazebo>
-    <!-- Gazebo Friction Overrides: Allows the 4 outer wheels to scrub/slide laterally -->
     <gazebo reference="left_wheel_one">
         <mu1>0.01</mu1>

Commit message: fix imu position

File: src/auracle_description/urdf/camera.xacro (robot description, xacro)
@@ -5,8 +5,10 @@
         <color rgba="1 0 0 1"/>
     </material>
+    <!-- x = chassis_length (0.3), i.e. flush with the front face, so the
+         chassis body itself doesn't clip the bottom of the camera's FOV -->
     <joint name="camera_joint" type="fixed">
         <parent link="chassis"/>
         <child link="camera_link"/>
-        <origin xyz="0.24 0 0.06" rpy="0 0 0"/>
+        <origin xyz="0.3 0 0.06" rpy="0 0 0"/>
     </joint>
     <link name="camera_link">

File: src/auracle_description/urdf/imu.xacro (robot description, xacro)
@@ -1,9 +1,8 @@
 <?xml version="1.0"?>
 <robot xmlns:xacro="http://www.ros.org/wiki/xacro" >
-    <!-- Adjust xyz to wherever the MPU6050 breakout actually sits on the chassis -->
     <joint name="imu_joint" type="fixed">
         <parent link="chassis"/>
         <child link="imu_link"/>
-        <origin xyz="0 0 0.05" rpy="0 0 0"/>
+        <origin xyz="0.15 0 0.05" rpy="0 0 0"/>
     </joint>
     <link name="imu_link">

File: src/auracle_description/urdf/robot_core.xacro (robot description, xacro)
@@ -57,21 +57,12 @@
         <material>Gazebo/Orange</material>
     </gazebo>
-    <!-- Rocker-to-chassis pivot. This has to be a real joint, not fixed:
-         it's the main degree of freedom that lets the whole rocker arm
-         (and everything hanging off it) rock forward/back as the wheels
-         cross terrain, instead of forcing the chassis to satisfy an
-         over-constrained rigid geometry. Passive (no actuator, not in
-         ros2_control) - it's driven purely by ground contact forces, with
-         damping/friction added just for numerical settling. Axis "1 0 0"
-         here is expressed in this joint's own (already rotated by the
-         rpy below) frame, and corresponds to the robot's lateral/pitch
-         axis - the correct axis for a suspension arm to rock about. -->
-    <joint name="left_wheel_rocker_joint" type="revolute">
+    <!-- Rocker-to-chassis pivot. TEMPORARILY fixed (rigid) while the
+         drooping-at-that-one-section issue is set aside - see the same
+         note on right_wheel_rocker_joint below for the revolute version
+         to restore once that's sorted. -->
+    <joint name="left_wheel_rocker_joint" type="fixed">
         <parent link="base_link"/>
         <child link="left_rocker"/>
         <origin xyz="${chassis_length/2} ${chassis_width/2+rocker_width/2} 0" rpy="0 0 ${pi/2}" />
-        <axis xyz="1 0 0"/>
-        <limit lower="-0.6" upper="0.6" effort="50" velocity="5"/>
-        <dynamics damping="2.0" friction="0.1"/>
     </joint>
     <link name="left_rocker">
@@ -121,17 +112,9 @@
         </xacro:inertial_box>
     </link>
-    <!-- Bogie pivot: on a real rocker-bogie, the two rear wheels per side
-         don't bolt straight onto the rocker - they hang off a small bogie
-         arm that itself pivots on the rocker, so those two wheels
-         equalize load on their own instead of forcing the rocker (and the
-         chassis above it) to twist to reach them both. Passive, same
-         reasoning as the rocker-to-chassis joint above. -->
-    <joint name="left_bogie_joint" type="revolute">
+    <!-- Bogie pivot: TEMPORARILY fixed, see left_wheel_rocker_joint above. -->
+    <joint name="left_bogie_joint" type="fixed">
         <parent link="left_rocker"/>
         <child link="left_bogie"/>
         <origin xyz="0 ${-rocker_length/2} 0" rpy="0 0 0" />
-        <axis xyz="1 0 0"/>
-        <limit lower="-0.4" upper="0.4" effort="50" velocity="5"/>
-        <dynamics damping="1.0" friction="0.1"/>
     </joint>
     <link name="left_bogie">
@@ -270,11 +253,21 @@
         <fdir1>1 0 0</fdir1>
     </gazebo>
-    <joint name="right_wheel_rocker_joint" type="revolute">
+    <!-- TEMPORARILY fixed - all 4 suspension joints (left/right rocker +
+         bogie) rigidified for now to rule out the suspension while
+         chasing the droop-at-one-section bug. To restore full
+         rocker-bogie articulation later, change type back to "revolute"
+         on all 4 and put back:
+           <axis xyz="1 0 0"/>
+           <limit lower="-0.6" upper="0.6" effort="50" velocity="5"/>   (rocker joints)
+           <limit lower="-0.4" upper="0.4" effort="50" velocity="5"/>   (bogie joints)
+           <dynamics damping="2.0" friction="0.1"/>                    (rocker joints)
+           <dynamics damping="1.0" friction="0.1"/>                    (bogie joints)
+         Rigidifying does mean the fixed 3-wheels-per-side frame will
+         fight ramp transitions again (see the wheel friction comment
+         below) - fine for flat-floor testing, revisit before ramps. -->
+    <joint name="right_wheel_rocker_joint" type="fixed">
         <parent link="base_link"/>
         <child link="right_rocker"/>
         <origin xyz="${chassis_length/2} ${-chassis_width/2-rocker_width/2} 0" rpy="0 0 ${pi/2}" />
-        <axis xyz="1 0 0"/>
-        <limit lower="-0.6" upper="0.6" effort="50" velocity="5"/>
-        <dynamics damping="2.0" friction="0.1"/>
     </joint>
     <link name="right_rocker">
@@ -319,11 +312,8 @@
         </xacro:inertial_box>
     </link>
-    <joint name="right_bogie_joint" type="revolute">
+    <joint name="right_bogie_joint" type="fixed">
         <parent link="right_rocker"/>
         <child link="right_bogie"/>
         <origin xyz="0 ${-rocker_length/2} 0" rpy="0 0 0" />
-        <axis xyz="1 0 0"/>
-        <limit lower="-0.4" upper="0.4" effort="50" velocity="5"/>
-        <dynamics damping="1.0" friction="0.1"/>
     </joint>
     <link name="right_bogie">
